File: pcb/yolochka-remastered/yolochka-remastered.kicad_pcb (KiCad board)
At the start: 2 copper layers, 241.5 x 80 mm, 109 parts, among them SW1 SW_PUSH, SW10 SW_PUSH, SW11 SW_PUSH, SW12 SW_PUSH, SW13 SW_PUSH, SW14 SW_PUSH, SW15 SW_PUSH, SW16 SW_PUSH, SW17 SW_PUSH, SW18 SW_PUSH, SW19 SW_PUSH, SW2 SW_PUSH, SW20 SW_PUSH, SW21 SW_PUSH, SW22 SW_PUSH, SW23 SW_PUSH, SW24 SW_PUSH, SW25 SW_PUSH, SW26 SW_PUSH, SW27 SW_PUSH, SW28 SW_PUSH, SW29 SW_PUSH, SW3 SW_PUSH, SW30 SW_PUSH, SW31 SW_PUSH, SW32 SW_PUSH, SW33 SW_PUSH, SW34 SW_PUSH, SW35 SW_PUSH, SW36 SW_PUSH, SW4 SW_PUSH, SW5 SW_PUSH, SW6 SW_PUSH, SW7 SW_PUSH, SW8 SW_PUSH, SW9 SW_PUSH, U1 ProMicro_r

Commit message: Change led position and initial reroute
Parts:
- moved D1 12.5 mm to (40.8, 62.0), turned to -60 degrees
- moved D10 12.5 mm to (240.2, 62.0), turned to -60 degrees
- moved D11 12.5 mm to (36.0, 81.0), turned to -60 degrees
- moved D12 12.5 mm to (55.0, 81.0), turned to -60 degrees
- moved D13 12.5 mm to (74.0, 81.0), turned to -60 degrees
- moved D14 12.5 mm to (93.0, 81.0), turned to -60 degrees
- moved D15 12.5 mm to (112.0, 81.0), turned to -60 degrees
- moved D16 12.5 mm to (169.0, 81.0), turned to -60 degrees
- moved D17 12.5 mm to (188.0, 81.0), turned to -60 degrees
- moved D18 12.5 mm to (207.0, 81.0), turned to -60 degrees
- moved D19 12.5 mm to (226.0, 81.0), turned to -60 degrees
- moved D2 12.5 mm to (59.8, 62.0), turned to -60 degrees
- moved D20 12.5 mm to (245.0, 81.0), turned to -60 degrees
- moved D21 12.5 mm to (31.2, 100.0), turned to -60 degrees
- moved D22 12.5 mm to (50.2, 100.0), turned to -60 degrees
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Routing:
- net GND: track 206.2 -> 0.00 mm
- net VCC: track 634.0 -> 798.1 mm
- net C0: track 349.0 -> 275.8 mm
- net C1: track 309.3 -> 237.4 mm
- net C2: track 274.7 -> 203.2 mm
- net R3: track 152.1 -> 90.0 mm, vias 3 -> 0
- net C4: track 175.7 -> 115.6 mm
- net C3: track 210.9 -> 153.8 mm
- net R2: track 133.1 -> 92.2 mm, vias 3 -> 1
- net Net-(LED30-DIN): track 89.5 -> 54.1 mm
- net Net-(LED1-DOUT): track 34.9 -> 0.00 mm
- net R4: track 153.8 -> 133.5 mm
- net Net-(LED10-DIN): track 41.1 -> 22.1 mm
- net C5: track 140.6 -> 123.3 mm
- net LED: track 13.9 -> 0.00 mm
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
Commit message: Initial route
Parts:
- added J1: ~, yolochka:FFC_CMD_1x20_P0.5mm, F.Cu at (150.0, 110.1)
Routing:
- net C4: track 115.6 -> 246.2 mm
- net C2: track 203.2 -> 332.8 mm
- net C3: track 153.8 -> 283.2 mm
- net R0: track 152.7 -> 262.8 mm
- net R1: track 130.4 -> 227.4 mm
- net C1: track 237.4 -> 328.1 mm
- net C0: track 275.8 -> 366.3 mm
- net R2: track 92.2 -> 178.0 mm
- net R5: track 154.4 -> 240.1 mm
- net R4: track 133.5 -> 207.6 mm
- net R3: track 90.0 -> 146.9 mm
- net C5: track 123.3 -> 145.4 mm
- net Net-(LED33-DOUT): track 33.2 -> 34.0 mm
Other:
- outline, holes or cut-outs redrawn

Commit message: Mostly routed
Parts:
- removed J1: ~, yolochka:FFC_CMD_1x20_P0.5mm
- turned LED1 to 0 degrees
- turned LED10 to 0 degrees
- turned LED2 to 0 degrees
- turned LED21 to 0 degrees
- turned LED22 to 0 degrees
- turned LED23 to 0 degrees
- turned LED24 to 0 degrees
- turned LED25 to 0 degrees
- turned LED26 to 0 degrees
- turned LED27 to 0 degrees
- turned LED28 to 0 degrees
- turned LED29 to 0 degrees
- turned LED3 to 0 degrees
- turned LED30 to 0 degrees
- turned LED4 to 0 degrees
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Routing:
- net C4: track 246.2 -> 871.5 mm, vias 8 -> 6
- net VCC: track 798.1 -> 1402.0 mm, vias 0 -> 2
- net C3: track 283.2 -> 758.5 mm, vias 8 -> 6
- net R5: track 240.1 -> 709.2 mm, vias 2 -> 0
- net C5: track 145.4 -> 597.0 mm
- net LED: track 0.00 -> 440.0 mm
- net C2: track 332.8 -> 648.9 mm, vias 8 -> 6
- net R0: track 262.8 -> 557.2 mm, vias 2 -> 0
- net R4: track 207.6 -> 460.0 mm, vias 2 -> 0
- net C1: track 328.1 -> 539.4 mm, vias 8 -> 6
- net R1: track 227.4 -> 335.9 mm, vias 2 -> 0
- net R3: track 146.9 -> 249.7 mm
- net Net-(LED21-DOUT): track 71.5 -> 0.00 mm
- net R2: track 178.0 -> 244.4 mm, vias 1 -> 0
- net C0: track 366.3 -> 422.2 mm, vias 8 -> 6
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Other:
- board size 241.5 x 80 mm -> 245.5 x 80 mm

Commit message: Switches routed, rgb led almost
Routing:
- net Net-(LED33-DOUT): track 0.00 -> 492.0 mm, vias 0 -> 6
- net VCC: track 1402.0 -> 952.3 mm, vias 2 -> 8
- net Net-(LED15-DOUT): track 0.00 -> 212.9 mm, vias 0 -> 2
- net Net-(LED21-DOUT): track 0.00 -> 80.4 mm, vias 0 -> 2
- net Net-(LED30-DIN): track 0.00 -> 79.7 mm, vias 0 -> 2
- net GND: track 0.00 -> 53.0 mm
- net Net-(LED1-DOUT): track 0.00 -> 44.3 mm, vias 0 -> 2
- net unconnected-(U1-RAW-Pad24): track 0.00 -> 33.3 mm
- net LED: track 440.0 -> 473.4 mm, vias 0 -> 1
- net C0: track 422.2 -> 454.9 mm
- net unconnected-(U1-GND-Pad23): track 0.00 -> 30.6 mm
- net unconnected-(U1-D2/RX1-Pad2): track 0.00 -> 30.6 mm
- net unconnected-(U1-RST-Pad22): track 0.00 -> 27.9 mm
- net R3: track 249.7 -> 276.6 mm, vias 0 -> 1
- net (no net): track 0.00 -> 23.0 mm
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
Commit message: Elements added, alsmost full routed
Parts:
- added LED37: YS-SK6812MINI-E, yolochka:YS-SK6812MINI-E_single, F.Cu at (228.8, 138.4)
- added LED38: YS-SK6812MINI-E, yolochka:YS-SK6812MINI-E_single, F.Cu at (236.2, 139.5)
- added LED39: YS-SK6812MINI-E, yolochka:YS-SK6812MINI-E_single, F.Cu at (225.1, 151.9)
- added LED40: YS-SK6812MINI-E, yolochka:YS-SK6812MINI-E_single, F.Cu at (232.5, 152.9)
- added LED41: YS-SK6812MINI-E, yolochka:YS-SK6812MINI-E_single, F.Cu at (239.9, 154.0)
- added PSW1: SW_SPDT, yolochka:MSK-12C02, F.Cu at (165.0, 45.0)
- added TP1: TestPoint_2Pole, yolochka:battery_conn_duplex, F.Cu at (169.7, 39.9)
- moved U1 5.50 mm to (150.0, 61.3)
Connections:
- U1 pad 2: unconnected-(U1-D2/RX1-Pad2) -> STATUS_LEDP
- U1 pad 23: unconnected-(U1-GND-Pad23) -> Net-(TP1-Pad1)
- U1 pad 24: unconnected-(U1-RAW-Pad24) -> VBAT
Routing:
- net Net-(LED16-DIN): track 1.35 -> 203.7 mm, vias 1 -> 2
- net VCC: track 952.3 -> 1007.2 mm, vias 8 -> 10
- net Net-(LED10-DIN): track 0.00 -> 43.7 mm, vias 0 -> 2
- net VBAT: track 0.00 -> 38.8 mm
- net R1: track 339.7 -> 376.1 mm, vias 1 -> 2
- net STATUS_LEDP: track 0.00 -> 36.1 mm
- net Net-(TP1-Pad1): track 0.00 -> 36.1 mm
- net unconnected-(U1-RAW-Pad24): track 33.3 -> 0.00 mm
- net unconnected-(U1-GND-Pad23): track 30.6 -> 0.00 mm
- net unconnected-(U1-D2/RX1-Pad2): track 30.6 -> 0.00 mm
- net R0: track 567.0 -> 595.9 mm, vias 1 -> 2
- net R2: track 260.0 -> 282.7 mm, vias 1 -> 2
- net C0: track 454.9 -> 474.5 mm, vias 6 -> 7
- net R5: track 700.3 -> 712.7 mm, vias 1 -> 2
- net GND: track 53.0 -> 64.0 mm
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Other:
- board size 245.5 x 80 mm -> 245.5 x 85.5 mm

Commit message: All things routed
Parts:
- added RSW1: SW_PUSH, yolochka:SW_EVQP7C01K, F.Cu at (135.0, 46.5)
- added U2: ~, yolochka:rgb3pin, F.Cu at (157.1, 82.5)
- added U3: ~, yolochka:rgb3pin, F.Cu at (231.1, 126.2)
- moved TP1 70.4 mm to (150.0, 107.5)
- moved LED38 18.5 mm to (234.8, 121.0)
- moved LED37 18.5 mm to (227.4, 120.0)
- moved LED39 18.5 mm to (223.7, 133.5), turned to -90 degrees
- moved LED40 18.5 mm to (231.1, 134.5), turned to -90 degrees
- moved LED41 18.5 mm to (238.5, 135.5)
Connections:
- LED40 pad 4: STATUS_LED -> STATUS_LEDS
- U1 pad 2: STATUS_LEDP -> STATUS_LED
- U1 pad 22: unconnected-(U1-RST-Pad22) -> reset
Routing:
- net VCC: track 1007.2 -> 1107.9 mm, vias 10 -> 11
- net R0: track 595.9 -> 673.5 mm
- net Net-(PSW1-B): track 0.00 -> 75.9 mm, vias 0 -> 1
- net R1: track 376.1 -> 450.5 mm
- net R2: track 282.7 -> 347.8 mm
- net LED: track 482.6 -> 544.2 mm
- net VCCS: track 0.00 -> 40.7 mm
- net C1: track 552.6 -> 592.3 mm
- net C2: track 662.2 -> 700.2 mm
- net R4: track 480.9 -> 517.7 mm, vias 2 -> 0
- net C3: track 771.5 -> 808.1 mm
- net STATUS_LEDP: track 36.1 -> 0.00 mm
- net unconnected-(U1-RST-Pad22): track 33.4 -> 0.00 mm
- net STATUS_LED: track 0.00 -> 30.7 mm
- net C4: track 893.6 -> 922.9 mm
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- added copper zone on B.Cu, net GNDS
- added copper zone on F.Cu, net GNDS
Other:
- board size 245.5 x 85.5 mm -> 245.5 x 95 mm
