File: pcb/yolochka-remastered/yolochka-remastered.kicad_sch (KiCad schematic)
At the start: 109 parts, among them SW1 SW_PUSH, SW10 SW_PUSH, SW11 SW_PUSH, SW12 SW_PUSH, SW13 SW_PUSH, SW14 SW_PUSH, SW15 SW_PUSH, SW16 SW_PUSH, SW17 SW_PUSH, SW18 SW_PUSH, SW19 SW_PUSH, SW2 SW_PUSH, SW20 SW_PUSH, SW21 SW_PUSH, SW22 SW_PUSH, SW23 SW_PUSH, SW24 SW_PUSH, SW25 SW_PUSH, SW26 SW_PUSH, SW27 SW_PUSH, SW28 SW_PUSH, SW29 SW_PUSH, SW3 SW_PUSH, SW30 SW_PUSH, SW31 SW_PUSH, SW32 SW_PUSH, SW33 SW_PUSH, SW34 SW_PUSH, SW35 SW_PUSH, SW36 SW_PUSH, SW4 SW_PUSH, SW5 SW_PUSH, SW6 SW_PUSH, SW7 SW_PUSH, SW8 SW_PUSH, SW9 SW_PUSH, U1 ProMicro_r

Commit message: Initial route
Parts:
- added J1: ~, yolochka:FFC_CMD_1x20_P0.5mm, symbol yolochka:CONN_01x20
Changed lines of the file:
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@@
+	)
+	(symbol
+		(lib_id "yolochka:CONN_01x20")
+		(at 264.16 295.91 0)
+		(unit 1)
+		(exclude_from_sim no)
+		(in_bom yes)
+		(on_board yes)
+		(dnp no)
+		(fields_autoplaced yes)
+		(property "Reference" "J1"
+			(at 265.43 297.1799 0)
+			(effects
+				(font
+					(size 1.27 1.27)
+				)
+				(justify left)
+			)
+		)
+		(property "Value" "~"
+			(at 264.16 323.85 0)
+			(effects
+				(font
+					(size 1.27 1.27)
+				)
+				(hide yes)
+			)
+		)
+		(property "Footprint" "yolochka:FFC_CMD_1x20_P0.5mm"
+			(at 264.16 295.91 0)
+			(effects
+				(font
+					(size 1.27 1.27)
+				)
+				(hide yes)
+			)
+		)
+		(property "Datasheet" ""
+			(at 264.16 295.91 0)
+			(effects
+				(font
+					(size 1.27 1.27)
+				)
+				(hide yes)
+			)
+		)
+		(property "Description" ""
+			(at 264.16 295.91 0)
+			(effects
+				(font
+					(size 1.27 1.27)
+				)
+				(hide yes)
+			)
+		)
+		(pin "3"
+		)
+		(pin "2"
+		)
+		(pin "1"
+		)
+		(pin "12"
+		)
+		(pin "15"
+		)
+		(pin "20"
+		)
+		(pin "4"
+		)
+		(pin "7"
+		)
+		(pin "10"
+		)
+		(pin "19"
+		)
+		(pin "13"
+		)
+		(pin "17"
+		)
+		(pin "6"
+		)
+		(pin "5"
+		)
+		(pin "11"
+		)
+		(pin "14"
+		)
+		(pin "18"
+		)
+		(pin "9"
+		)
+		(pin "8"
+		)
+		(pin "16"
+		)
+		(instances
+			(project ""
+				(path "/f379e286-fd5d-4a21-8f59-85bfb7393b03"
+					(reference "J1")
+					(unit 1)
+				)
+			)
+		)
 	)
 	(symbol

Commit message: Elements added, alsmost full routed
Parts:
- removed J1: ~, yolochka:FFC_CMD_1x20_P0.5mm, symbol yolochka:CONN_01x20
- added LED37, LED38, LED39, LED40, LED41: YS-SK6812MINI-E, yolochka:YS-SK6812MINI-E_single, symbol yolochka:YS-SK6812MINI-E_v2
- added PSW1: SW_SPDT, yolochka:MSK-12C02, symbol yolochka:SW_SPDT
- added TP1: TestPoint_2Pole, yolochka:battery_conn_duplex, symbol Connector:TestPoint_2Pole
Connections:
- net STATUS_LEDP: now reaches U1.2 (D2/RX1)
- net at U1.23 (GND): now also TP1.1
- net VBAT: now reaches U1.24 (RAW)
- net VBAT: now also PSW1.1 (A)
- new net: LED37.2 (DOUT), LED38.4 (DIN)
- new net: LED37.4 (DIN), LED39.2 (DOUT)
- new net: LED38.2 (DOUT), LED41.4 (DIN)
- new net: LED39.4 (DIN), LED40.2 (DOUT)
- new net: PSW1.2 (B), TP1.2
- new net GNDS: LED37.3 (GND), LED38.3 (GND), LED39.3 (GND), LED40.3 (GND), LED41.3 (GND)
- new net STATUS_LED: LED40.4 (DIN)
- new net VCCS: LED37.1 (VDD), LED38.1 (VDD), LED39.1 (VDD), LED40.1 (VDD), LED41.1 (VDD)
- no-connect marks 1 -> 7
Other:
- moved on the sheet: U1

Commit message: All things routed
Parts:
- added RSW1: SW_PUSH, yolochka:SW_EVQP7C01K, symbol yolochka:SW_PUSH
- added U2, U3: ~, yolochka:rgb3pin, symbol yolochka:rgb3pin
Connections:
- net STATUS_LEDP is gone; now on net STATUS_LED: U1.2 (D2/RX1)
- net GND: now also RSW1.2, U2.1 (GND)
- net GNDS: now also U3.1 (GND)
- net STATUS_LED: now also U2.3 (LED); no longer LED40.4 (DIN)
- net VCC: now also U2.2 (VCC)
- net VCCS: now also U3.2 (VCC)
- net reset: now reaches U1.22 (RST)
- net reset: now also RSW1.1
- new net STATUS_LEDS: LED40.4 (DIN), U3.3 (LED)
